File: fishsensor.sch (KiCad schematic (older format))
At the start: 1 part

Commit message: 2021-11-04
Parts:
- added C1, C10, C11, C12, C2, C4, C5, C7, C9: 0.1u, Capacitor_SMD:C_0603_1608Metric, symbol Device:C
- added C3, C6: 0.01u, Capacitor_SMD:C_0603_1608Metric, symbol Device:C
- added C8: 2.2n, Capacitor_SMD:C_0603_1608Metric, symbol Device:C
- added D1, D2: LED_Dual_ACA, LED_THT:LED_D5.0mm-3, symbol Device:LED_Dual_ACA
- added J1: Li-Po, tp:boot, symbol Connector_Generic:Conn_01x02
- added J2: UART, Connector_PinHeader_2.54mm:PinHeader_1x03_P2.54mm_Vertical, symbol Connector_Generic:Conn_01x03
- added J3: USB_B_Micro, Connector_USB:USB_Micro-B_GCT_USB3076-30-A, symbol Connector:USB_B_Micro
- added Q1, Q2: BC856B,215, Package_TO_SOT_SMD:SOT-23, symbol Device:Q_PNP_BEC
- added R1, R11, R4, R5, R6, R7: 10k, Resistor_SMD:R_0603_1608Metric, symbol Device:R
- added R10: 2k, Resistor_SMD:R_0603_1608Metric, symbol Device:R
- added R12, R13: 33k, Resistor_SMD:R_0603_1608Metric, symbol Device:R
- added R14: 1k, Resistor_SMD:R_0603_1608Metric, symbol Device:R
- added R2, R3, R8, R9: 510, Resistor_SMD:R_0603_1608Metric, symbol Device:R
- added SW1: boot, Button_Switch_SMD:SW_Push_SPST_NO_Alps_SKRK, symbol Switch:SW_Push
- added SW2: pwr, Button_Switch_SMD:SW_Push_SPST_NO_Alps_SKRK, symbol Switch:SW_Push
- added U1: MIC5318-3.3YD5-TR, Package_TO_SOT_SMD:TSOT-23-5, symbol MIC531833YD5TR:MIC5318-3.3YD5-TR
- added U3: MPU-6050, Sensor_Motion:InvenSense_QFN-24_4x4mm_P0.5mm, symbol Sensor_Motion:MPU-6050
- added U4: MCP73831-2-OT, Package_TO_SOT_SMD:SOT-23-5, symbol Battery_Management:MCP73831-2-OT
- gave numbers to parts that had none: 1
Connections:
- net Earth: now reaches U2.1 (GND), U2.15 (GND), U2.38 (GND), U2.39 (GND)
- net Earth: now also C1.2, C10.2, C11.2, C12.1, C2.2, C3.1, C4.2, C5.1, C6.2, C7.1, C8.1, C9.2, D1.2 (K), D2.2 (K), J1.2 (Pin_2), J2.1 (Pin_1), J3.5 (GND), J3.6 (Shield), R10.2, R6.2, R7.2, SW1.1, U1.2 (GND), U3.1 (CLKIN), U3.18 (GND), U4.2 (VSS)
- net BTN: now reaches U2.12 (IO27)
- net BTN: now also R14.2
- net +3V3: now reaches U2.2 (VDD)
- net +3V3: now also C4.1, C5.2, C6.1, Q1.2 (E), Q2.2 (E), R1.2, R11.1, R4.1, R5.1, SW2.1, U1.5 (OUT), U3.13 (VDD), U3.8 (VDDIO)
- net BOOT: now reaches U2.25 (IO0)
- net BOOT: now also C1.1, R1.1, SW1.2
- net EN: now reaches U2.3 (EN)
- net EN: now also C10.1, R11.2
- net LED_RED: now reaches U2.30 (IO18)
- net LED_RED: now also R13.2
- net LED_GRN: now reaches U2.31 (IO19)
- net LED_GRN: now also R2.1, R8.1
- net SDA: now reaches U2.33 (IO21)
- net SDA: now also R5.2, U3.24 (SDA)
- net RX: now reaches U2.34 (RXD0/IO3)
- net RX: now also J2.2 (Pin_2)
- net TX: now reaches U2.35 (TXD0/IO1)
- net TX: now also J2.3 (Pin_3)
- net SCL: now reaches U2.36 (IO22)
- net SCL: now also R4.2, U3.23 (SCL)
- net INT: now reaches U2.37 (IO23)
- net INT: now also U3.12 (INT)
- new net: C7.2, U3.10 (REGOUT)
- new net: R7.1, U3.11 (FSYNC)
- new net: C8.2, U3.20 (CPOUT)
- new net: R6.1, U3.9 (AD0)
- new net: C3.2, U1.4 (BYP)
- new net: D1.1 (A1), R2.2
- new net: Q1.3 (C), Q2.3 (C), R3.1, R9.1
- new net: D1.3 (A2), R3.2
- new net: D2.1 (A1), R8.2
- new net: D2.3 (A2), R9.2
- new net: C12.2, R14.1, SW2.2
- new net: R10.1, U4.5 (PROG)
- new net: Q1.1 (B), R12.1
- new net: Q2.1 (B), R13.1
- new net BATT: C2.1, C9.1, J1.1 (Pin_1), U1.1 (IN), U1.3 (EN), U4.3 (VBAT)
- new net CHRG: R12.2, U4.1 (STAT)
- new net VBUS: C11.1, J3.1 (VBUS), U4.4 (VDD)
- no-connect marks 0 -> 4
Other:
- moved on the sheet: U2
